File: lightstrip/lightstrip.kicad_pcb (KiCad board)
At the start: 2 copper layers, 19 parts, among them J1 Connector

Commit message: Spread strip to 9".
Parts:
- added H1: MountingHole, MountingHole:MountingHole_2.2mm_M2, F.Cu at (25.4, 61.0)
- added H2: MountingHole, MountingHole:MountingHole_2.2mm_M2, F.Cu at (246.4, 61.0)
- moved D1 65.6 mm to (104.2, 60.9), turned to 0 degrees
- moved D5 64.2 mm to (170.8, 60.9), turned to 0 degrees
- moved D7 62.9 mm to (238.2, 60.9), turned to 0 degrees
- moved D18 48.8 mm to (183.6, 61.0), turned to 0 degrees
- moved D16 47.0 mm to (116.9, 60.9), turned to 0 degrees
- moved D14 45.0 mm to (50.2, 61.0), turned to 0 degrees
- moved D4 43.9 mm to (93.4, 61.0), turned to 0 degrees
- moved D6 42.0 mm to (160.1, 61.0), turned to 0 degrees
- moved D8 40.7 mm to (227.4, 60.9), turned to 0 degrees
- moved D17 26.6 mm to (194.3, 61.0), turned to 0 degrees
- moved D15 24.7 mm to (127.7, 60.9), turned to 0 degrees
- moved D3 22.8 mm to (61.0, 61.0), turned to 0 degrees
- moved D2 21.6 mm to (82.6, 61.0), turned to 0 degrees
- moved D10 19.8 mm to (149.3, 60.9), turned to 0 degrees
- moved D12 18.5 mm to (216.6, 60.9), turned to 0 degrees
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Connections:
- J1 pad 3: /warm1 -> /warm3
- J1 pad 4: /cool1 -> /warm2
- J1 pad 5: /warm2 -> /cool3
- J1 pad 7: /warm3 -> /warm1
- J1 pad 8: /cool3 -> /cool1
Routing:
- net +12V: track 5.28 -> 0.00 mm, vias 3 -> 0

Commit message: More layout.
Parts:
- moved D10 51.4 mm to (167.0, 109.2)
- moved D11 51.4 mm to (156.2, 109.2)
- moved D12 51.4 mm to (234.4, 109.2)
- moved D15 51.4 mm to (145.5, 109.2)
- moved D16 51.4 mm to (134.7, 109.2)
- moved D5 51.4 mm to (188.6, 109.2)
- moved D7 51.4 mm to (255.9, 109.2)
- moved D8 51.4 mm to (245.2, 109.2)
- moved H2 51.4 mm to (264.2, 109.2)
- moved D13 51.4 mm to (222.9, 109.2)
- moved D14 51.4 mm to (68.0, 109.2)
- moved D17 51.4 mm to (212.1, 109.2)
- moved D18 51.4 mm to (201.3, 109.2)
- moved D2 51.4 mm to (100.4, 109.2)
- moved D3 51.4 mm to (78.8, 109.2)
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Routing:
- net /warm3: track 0.00 -> 161.0 mm, vias 0 -> 2
- net /cool3: track 0.00 -> 146.9 mm, vias 0 -> 2
- net /warm2: track 0.00 -> 94.3 mm, vias 0 -> 2
- net /cool2: track 0.00 -> 80.8 mm, vias 0 -> 2
- net Net-(D13-Pad2): track 0.00 -> 21.9 mm
- net Net-(D12-Pad1): track 0.00 -> 21.8 mm
- net Net-(D11-Pad1): track 0.00 -> 21.2 mm
- net Net-(D10-Pad1): track 0.00 -> 21.2 mm
- net Net-(D4-Pad1): track 0.00 -> 21.2 mm
- net Net-(D14-Pad2): track 0.00 -> 21.2 mm
- net Net-(D12-Pad2): track 0.00 -> 21.2 mm
- net Net-(D11-Pad2): track 0.00 -> 21.2 mm
- net Net-(D1-Pad1): track 0.00 -> 21.2 mm
- net Net-(D2-Pad1): track 0.00 -> 21.2 mm
- net Net-(D13-Pad1): track 0.00 -> 21.1 mm
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Other:
- board outline added: 228.6 x 7.6 mm
